File: Aamber Pegasus Replica v1.5.sch (KiCad schematic (older format))
At the start: 123 parts, among them IC1 74LS14, IC11 74LS245, IC12 74LS241, IC12 MC6809, IC13 74LS241, IC14 74LS139, IC15 74LS139, IC16 74LS139, IC17 74LS08, IC18 TMS2532, IC19 6821, IC19 TMS2532, IC2 74LS32, IC20 TMS2532, IC21 6821, IC22 74LS20, IC23 MC2114RAM, IC24 MC2114RAM, IC25 MC2114RAM, IC26 MC2114RAM, IC27 MC2114RAM, IC28 MC2114RAM, IC3 74LS00, IC30 74LS245, IC31 MC2114RAM, IC32 MC2114RAM, IC33 74LS86, IC34 MC2114RAM, IC35 MC2114RAM, IC36 MC66710, IC37 MC2114RAM, IC38 MC2114RAM, IC39 74LS157, IC4 74LS21, IC40 74LS165, IC41 74LS157, IC42 74LS245, IC43 74LS04, IC45 74LS157, IC46 74LS74, IC47 74LS32, IC5 74LS123, IC6 74LS74, IC7 74LS93, IC8 74LS93, IC9 74LS04, SW1 RESET SWITCH, X1 4MHz

Commit message: Replaced rescue components with Aamber.lib components
- Removed rescue and cache libs from revision control (they are auto-generated).

- Replaced references to rescue lib from schematic, and replaced with same
references to Aamber.lib.
Parts:
- IC18, IC19, IC20: symbol Aamber-Pegasus-Replica-v1.5-rescue:TMS2532-Aamber -> Aamber:TMS2532
- IC23, IC24, IC25, IC26, IC27, IC28, IC31, IC32, IC34, IC35, IC37, IC38: symbol Aamber-Pegasus-Replica-v1.5-rescue:MC2114RAM-Aamber -> Aamber:MC2114RAM
- IC36: symbol Aamber-Pegasus-Replica-v1.5-rescue:MC66710-Aamber -> Aamber:MC66710
- UIC44: symbol Aamber-Pegasus-Replica-v1.5-rescue:MC14066-Aamber -> Aamber:MC14066
Changed lines of the file:
@@
 50HERTZ
 $Comp
-L Aamber-Pegasus-Replica-v1.5-rescue:MC2114RAM-Aamber IC25
+L Aamber:MC2114RAM IC25
 U 1 1 5E6FDFAA
 P 4500 19250
@@
 $EndComp
 $Comp
-L Aamber-Pegasus-Replica-v1.5-rescue:MC2114RAM-Aamber IC27
+L Aamber:MC2114RAM IC27
 U 1 1 5E75CD16
 P 4500 21550
@@
 $EndComp
 $Comp
-L Aamber-Pegasus-Replica-v1.5-rescue:MC2114RAM-Aamber IC26
+L Aamber:MC2114RAM IC26
 U 1 1 5E75E6DC
 P 7500 19200
@@
 $EndComp
 $Comp
-L Aamber-Pegasus-Replica-v1.5-rescue:MC2114RAM-Aamber IC28
+L Aamber:MC2114RAM IC28
 U 1 1 5E75E6E6
 P 7500 21500
@@
 D7
 $Comp
-L Aamber-Pegasus-Replica-v1.5-rescue:MC2114RAM-Aamber IC37
+L Aamber:MC2114RAM IC37
 U 1 1 5E8D23AE
 P 19650 25250
@@
 $EndComp
 $Comp
-L Aamber-Pegasus-Replica-v1.5-rescue:MC2114RAM-Aamber IC32
+L Aamber:MC2114RAM IC32
 U 1 1 5E98E810
 P 22000 20050
@@
 	23150 20150 22500 20150
 $Comp
-L Aamber-Pegasus-Replica-v1.5-rescue:MC2114RAM-Aamber IC31
+L Aamber:MC2114RAM IC31
 U 1 1 5E98E80A
 P 19600 20000
@@
 	23700 22550 23950 22550
 $Comp
-L Aamber-Pegasus-Replica-v1.5-rescue:MC66710-Aamber IC36
+L Aamber:MC66710 IC36
 U 1 1 723C7D41
 P 16900 24900
@@
 Connection ~ 18250 24750
 $Comp
-L Aamber-Pegasus-Replica-v1.5-rescue:MC2114RAM-Aamber IC38
+L Aamber:MC2114RAM IC38
 U 1 1 7487509C
 P 21950 25250
@@
 	20150 22650 20150 23750
 $Comp
-L Aamber-Pegasus-Replica-v1.5-rescue:MC2114RAM-Aamber IC34
+L Aamber:MC2114RAM IC34
 U 1 1 5E8CE72A
 P 19650 22550
@@
 	41800 20300 39900 20300
 $Comp
-L Aamber-Pegasus-Replica-v1.5-rescue:MC14066-Aamber UIC44
+L Aamber:MC14066 UIC44
 U 1 1 60746A6C
 P 40800 21600
@@
 	4000 21050 3200 21050
 $Comp
-L Aamber-Pegasus-Replica-v1.5-rescue:MC2114RAM-Aamber IC24
+L Aamber:MC2114RAM IC24
 U 1 1 5E75E6D2
 P 7500 17100
@@
 $EndComp
 $Comp
-L Aamber-Pegasus-Replica-v1.5-rescue:MC2114RAM-Aamber IC23
+L Aamber:MC2114RAM IC23
 U 1 1 5E5E3975
 P 4500 17150
@@
 	22450 22650 22950 22650
 $Comp
-L Aamber-Pegasus-Replica-v1.5-rescue:MC2114RAM-Aamber IC35
+L Aamber:MC2114RAM IC35
 U 1 1 5E8D033D
 P 21950 22550
@@
 	37350 7750 37450 7850
 $Comp
-L Aamber-Pegasus-Replica-v1.5-rescue:TMS2532-Aamber IC20
+L Aamber:TMS2532 IC20
 U 1 1 5FA70CA2
 P 35850 9900
@@
 $EndComp
 $Comp
-L Aamber-Pegasus-Replica-v1.5-rescue:TMS2532-Aamber IC19
+L Aamber:TMS2532 IC19
 U 1 1 5FB0DA67
 P 35850 6900
@@
 	37450 7250 40250 7250
 $Comp
-L Aamber-Pegasus-Replica-v1.5-rescue:TMS2532-Aamber IC18
+L Aamber:TMS2532 IC18
 U 1 1 5FBFC0B5
 P 35850 3850

Commit message: Revert "Replaced rescue components with Aamber.lib components"
This reverts commit 4ae101721c61db13dc762e7416d8930497a32c58.
Parts:
- IC18, IC19, IC20: symbol Aamber:TMS2532 -> Aamber-Pegasus-Replica-v1.5-rescue:TMS2532-Aamber
- IC23, IC24, IC25, IC26, IC27, IC28, IC31, IC32, IC34, IC35, IC37, IC38: symbol Aamber:MC2114RAM -> Aamber-Pegasus-Replica-v1.5-rescue:MC2114RAM-Aamber
- IC36: symbol Aamber:MC66710 -> Aamber-Pegasus-Replica-v1.5-rescue:MC66710-Aamber
- UIC44: symbol Aamber:MC14066 -> Aamber-Pegasus-Replica-v1.5-rescue:MC14066-Aamber
Changed lines of the file:
@@
 50HERTZ
 $Comp
-L Aamber:MC2114RAM IC25
+L Aamber-Pegasus-Replica-v1.5-rescue:MC2114RAM-Aamber IC25
 U 1 1 5E6FDFAA
 P 4500 19250
@@
 $EndComp
 $Comp
-L Aamber:MC2114RAM IC27
+L Aamber-Pegasus-Replica-v1.5-rescue:MC2114RAM-Aamber IC27
 U 1 1 5E75CD16
 P 4500 21550
@@
 $EndComp
 $Comp
-L Aamber:MC2114RAM IC26
+L Aamber-Pegasus-Replica-v1.5-rescue:MC2114RAM-Aamber IC26
 U 1 1 5E75E6DC
 P 7500 19200
@@
 $EndComp
 $Comp
-L Aamber:MC2114RAM IC28
+L Aamber-Pegasus-Replica-v1.5-rescue:MC2114RAM-Aamber IC28
 U 1 1 5E75E6E6
 P 7500 21500
@@
 D7
 $Comp
-L Aamber:MC2114RAM IC37
+L Aamber-Pegasus-Replica-v1.5-rescue:MC2114RAM-Aamber IC37
 U 1 1 5E8D23AE
 P 19650 25250
@@
 $EndComp
 $Comp
-L Aamber:MC2114RAM IC32
+L Aamber-Pegasus-Replica-v1.5-rescue:MC2114RAM-Aamber IC32
 U 1 1 5E98E810
 P 22000 20050
@@
 	23150 20150 22500 20150
 $Comp
-L Aamber:MC2114RAM IC31
+L Aamber-Pegasus-Replica-v1.5-rescue:MC2114RAM-Aamber IC31
 U 1 1 5E98E80A
 P 19600 20000
@@
 	23700 22550 23950 22550
 $Comp
-L Aamber:MC66710 IC36
+L Aamber-Pegasus-Replica-v1.5-rescue:MC66710-Aamber IC36
 U 1 1 723C7D41
 P 16900 24900
@@
 Connection ~ 18250 24750
 $Comp
-L Aamber:MC2114RAM IC38
+L Aamber-Pegasus-Replica-v1.5-rescue:MC2114RAM-Aamber IC38
 U 1 1 7487509C
 P 21950 25250
@@
 	20150 22650 20150 23750
 $Comp
-L Aamber:MC2114RAM IC34
+L Aamber-Pegasus-Replica-v1.5-rescue:MC2114RAM-Aamber IC34
 U 1 1 5E8CE72A
 P 19650 22550
@@
 	41800 20300 39900 20300
 $Comp
-L Aamber:MC14066 UIC44
+L Aamber-Pegasus-Replica-v1.5-rescue:MC14066-Aamber UIC44
 U 1 1 60746A6C
 P 40800 21600
@@
 	4000 21050 3200 21050
 $Comp
-L Aamber:MC2114RAM IC24
+L Aamber-Pegasus-Replica-v1.5-rescue:MC2114RAM-Aamber IC24
 U 1 1 5E75E6D2
 P 7500 17100
@@
 $EndComp
 $Comp
-L Aamber:MC2114RAM IC23
+L Aamber-Pegasus-Replica-v1.5-rescue:MC2114RAM-Aamber IC23
 U 1 1 5E5E3975
 P 4500 17150
@@
 	22450 22650 22950 22650
 $Comp
-L Aamber:MC2114RAM IC35
+L Aamber-Pegasus-Replica-v1.5-rescue:MC2114RAM-Aamber IC35
 U 1 1 5E8D033D
 P 21950 22550
@@
 	37350 7750 37450 7850
 $Comp
-L Aamber:TMS2532 IC20
+L Aamber-Pegasus-Replica-v1.5-rescue:TMS2532-Aamber IC20
 U 1 1 5FA70CA2
 P 35850 9900
@@
 $EndComp
 $Comp
-L Aamber:TMS2532 IC19
+L Aamber-Pegasus-Replica-v1.5-rescue:TMS2532-Aamber IC19
 U 1 1 5FB0DA67
 P 35850 6900
@@
 	37450 7250 40250 7250
 $Comp
-L Aamber:TMS2532 IC18
+L Aamber-Pegasus-Replica-v1.5-rescue:TMS2532-Aamber IC18
 U 1 1 5FBFC0B5
 P 35850 3850
