File: Aamber Pegasus Replica v1.5.sch (KiCad schematic (older format))
At the start: 123 parts, among them IC1 74LS14, IC11 74LS245, IC12 74LS241, IC12 MC6809, IC13 74LS241, IC14 74LS139, IC15 74LS139, IC16 74LS139, IC17 74LS08, IC18 TMS2532, IC19 6821, IC19 TMS2532, IC2 74LS32, IC20 TMS2532, IC21 6821, IC22 74LS20, IC23 MC2114RAM, IC24 MC2114RAM, IC25 MC2114RAM, IC26 MC2114RAM, IC27 MC2114RAM, IC28 MC2114RAM, IC3 74LS00, IC30 74LS245, IC31 MC2114RAM, IC32 MC2114RAM, IC33 74LS86, IC34 MC2114RAM, IC35 MC2114RAM, IC36 MC66710, IC37 MC2114RAM, IC38 MC2114RAM, IC39 74LS157, IC4 74LS21, IC40 74LS165, IC41 74LS157, IC42 74LS245, IC43 74LS04, IC45 74LS157, IC46 74LS74, IC47 74LS32, IC5 74LS123, IC6 74LS74, IC7 74LS93, IC8 74LS93, IC9 74LS04, SW1 RESET SWITCH, X1 4MHz

Commit message: Cleanups in progress.
Parts:
- IC18, IC19, IC20: symbol Memory_EPROM:TMS2532 -> Aamber:TMS2532
- IC23, IC24, IC25, IC26, IC27, IC28, IC31, IC32, IC34, IC35, IC37, IC38: symbol 74xx:MC2114RAM -> Aamber:MC2114RAM
- IC36: symbol Memory_EPROM:MC66710 -> Aamber:MC66710
- UIC44: symbol 74xx:MC14066 -> Aamber:MC14066
Connections:
- net labels removed: D0-D3, D4-D7
- wire segments 1259 -> 1280
Other:
- note removed: "What \nhappens here \n(to Pin 8 RAM??)"
- moved on the sheet: IC17C, IC17D, IC18, IC19, IC20, IC31, IC32, JP1, R?, UIC44

Commit message: Add names for wires and simplifiy
Parts:
- JP3: value JP3 -> Jumper
Connections:
- net labels added: B0-B7, CHAR-ROM, UA0, UA1, UA2, UA3, UA4, UA5, UA6, UA7, UB0, UB1, UB2, UB3, UB4, UB5, UB6, UB7
- wire segments 1280 -> 1296
Other:
- moved on the sheet: IC14A, IC14B, IC15A, IC15B, IC16A, IC16B, IC17C, IC17D, IC18, IC19, IC20, IC2A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

Commit message: Connecting all the ports
Parts:
- IC18, IC19, IC20: symbol Aamber:TMS2532 -> Aamber-Pegasus-Replica-v1.5-rescue:TMS2532-Aamber
- IC23, IC24, IC25, IC26, IC27, IC28, IC31, IC32, IC34, IC35, IC37, IC38: symbol Aamber:MC2114RAM -> Aamber-Pegasus-Replica-v1.5-rescue:MC2114RAM-Aamber
- IC36: symbol Aamber:MC66710 -> Aamber-Pegasus-Replica-v1.5-rescue:MC66710-Aamber
- UIC44: symbol Aamber:MC14066 -> Aamber-Pegasus-Replica-v1.5-rescue:MC14066-Aamber
Connections:
- net A10: no longer IC17.1, IC22.8, IC39.15 (E), IC41.15 (E), IC47.5
- new net X: IC17.1, IC22.8, IC39.15 (E), IC41.15 (E), IC47.5
Other:
- moved on the sheet: C1, C10, C2, C3, C4, C5, C6, C7, C8, C9, D1, D2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

Commit message: Connect all busses + some fixes
Connections:
- net ~SET is gone; now on net ~SEL: IC17.8
- net D0: now also IC19.33 (D0)
- net D1: now also IC19.32 (D1)
- net D2: now also IC19.31 (D2)
- net D3: now also IC19.30 (D3)
- net D4: now also IC19.29 (D4)
- net D5: now also IC19.28 (D5)
- net D6: now also IC19.27 (D6)
- net D7: now also IC19.26 (D7)
- net UA0: now also IC19.2 (PA0)
- net UA1: now also IC19.3 (PA1)
- net UA2: now also IC19.4 (PA2)
- net UA3: now also IC19.5 (PA3)
- net UA4: now also IC19.6 (PA4)
- net UA5: now also IC19.7 (PA5)
- net UA6: now also IC19.8 (PA6)
- net UA7: now also IC19.9 (PA7)
- net UB0: now also IC19.10 (PB0)
- net UB1: now also IC19.11 (PB1)
- net UB2: now also IC19.12 (PB2)
- net UB3: now also IC19.13 (PB3)
- net UB4: now also IC19.14 (PB4)
- net UB5: now also IC19.15 (PB5)
- net UB6: now also IC19.16 (PB6)
- net UB7: now also IC19.17 (PB7)
- net SET renamed ~SEL

Commit message: Revert "Connect all busses + some fixes"
This reverts commit 6c6519010b8e12310b57cd390e3bec1288484da7.
Connections:
- net D0: no longer IC19.33 (D0)
- net D1: no longer IC19.32 (D1)
- net D2: no longer IC19.31 (D2)
- net D3: no longer IC19.30 (D3)
- net D4: no longer IC19.29 (D4)
- net D5: no longer IC19.28 (D5)
- net D6: no longer IC19.27 (D6)
- net D7: no longer IC19.26 (D7)
- net UA0: no longer IC19.2 (PA0)
- net UA1: no longer IC19.3 (PA1)
- net UA2: no longer IC19.4 (PA2)
- net UA3: no longer IC19.5 (PA3)
- net UA4: no longer IC19.6 (PA4)
- net UA5: no longer IC19.7 (PA5)
- net UA6: no longer IC19.8 (PA6)
- net UA7: no longer IC19.9 (PA7)
- net UB0: no longer IC19.10 (PB0)
- net UB1: no longer IC19.11 (PB1)
- net UB2: no longer IC19.12 (PB2)
- net UB3: no longer IC19.13 (PB3)
- net UB4: no longer IC19.14 (PB4)
- net UB5: no longer IC19.15 (PB5)
- net UB6: no longer IC19.16 (PB6)
- net UB7: no longer IC19.17 (PB7)
- net ~SEL renamed SET
- net SET: no longer IC17.8
- new net ~SET: IC17.8

Commit message: Revert "Connecting all the ports"
This reverts commit 235e34fc1a66492c80c072c2703872a2e53422df.
Parts:
- IC18, IC19, IC20: symbol Aamber-Pegasus-Replica-v1.5-rescue:TMS2532-Aamber -> Aamber:TMS2532
- IC23, IC24, IC25, IC26, IC27, IC28, IC31, IC32, IC34, IC35, IC37, IC38: symbol Aamber-Pegasus-Replica-v1.5-rescue:MC2114RAM-Aamber -> Aamber:MC2114RAM
- IC36: symbol Aamber-Pegasus-Replica-v1.5-rescue:MC66710-Aamber -> Aamber:MC66710
- UIC44: symbol Aamber-Pegasus-Replica-v1.5-rescue:MC14066-Aamber -> Aamber:MC14066
Connections:
- net X is gone; now on net A10: IC17.1, IC22.8, IC39.15 (E), IC41.15 (E), IC47.5
Other:
- moved on the sheet: C1, C10, C2, C3, C4, C5, C6, C7, C8, C9, D1, D2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

Commit message: Moved individual pages into schematic subsheets for readability.
Parts:
- removed C1: 150nf, symbol Device:C
- removed C10: 1nf Disc Ceramic, symbol Device:C
- removed C2: 330nf, symbol Device:C
- removed C3: 100uf ceramic, symbol Device:C
- removed C4: 1uf 35v tantalum, symbol Device:C
- removed C5, C6: 27pf ceramic, symbol Device:C
- removed C7: 20nf ceramic, symbol Device:C
- removed C8: 100nf ceramic, symbol Device:C
- removed C9: 47pf Disc, symbol Device:C
- removed D1, D2, D3, D4, D5, D6, D7: IN4148, symbol pspice:DIODE
- removed unit 6 of IC1
- removed unit 5 of IC1
- removed unit 4 of IC1
- removed unit 1 of IC1
- removed unit 3 of IC1
- removed unit 2 of IC1
- removed IC11, IC30, IC42: 74LS245, symbol 74xx:74LS245
- removed IC12: MC6809, Package_DIP:DIP-40_W15.24mm, symbol CPU_NXP_6800:MC6809
- removed IC12, IC13: 74LS241, symbol 74xx:74LS241
- removed unit 1 of IC14
- removed unit 2 of IC14
- removed unit 1 of IC15
- removed unit 2 of IC15
- removed unit 1 of IC16
- removed unit 2 of IC16
- removed unit 3 of IC17
- removed unit 4 of IC17
- removed unit 1 of IC17
- removed unit 2 of IC17
- removed IC18, IC19, IC20: TMS2532, symbol Aamber:TMS2532
- removed IC19, IC21: 6821, Package_DIP:DIP-40_W15.24mm, symbol Interface:6821
- removed unit 2 of IC2
- removed unit 1 of IC2
- removed unit 4 of IC2
- removed unit 3 of IC2
- removed unit 2 of IC22
- removed unit 1 of IC22
- removed IC23, IC24, IC25, IC26, IC27, IC28, IC31, IC32, IC34, IC35, IC37, IC38: MC2114RAM, symbol Aamber:MC2114RAM
- removed unit 3 of IC3
- removed unit 4 of IC3
- removed unit 2 of IC3
- removed unit 3 of IC33
- removed unit 4 of IC33
- removed unit 1 of IC33
- removed unit 2 of IC33
- removed IC36: MC66710, symbol Aamber:MC66710
- removed IC39, IC41, IC45: 74LS157, symbol 74xx:74LS157
- removed unit 1 of IC4
- removed unit 2 of IC4
- removed IC40: 74LS165, symbol 74xx:74LS165
- removed IC43: 74LS04, symbol 74xx:74LS04
- removed unit 1 of IC46
- removed unit 2 of IC47
- removed unit 4 of IC47
- removed unit 1 of IC5
- removed unit 2 of IC5
- removed unit 1 of IC6
- removed unit 2 of IC6
- removed IC7, IC8: 74LS93, symbol 74xx:74LS93
- removed unit 3 of IC9
- removed unit 1 of IC9
- removed unit 4 of IC9
- removed unit 2 of IC9
- removed unit 5 of IC9
- removed unit 6 of IC9
- removed JP1, JP2, JP3: Jumper, symbol Device:Jumper
- removed R1, R2: 220K, symbol Device:R
- removed R10, R11, R12, R16, R17, R18, R19, R20, R21, R22, R23, R28, R29, R30, R31, R32, R33, R7, R8, R9, R? (x2): 1k, symbol Device:R
- removed R14: 470K, symbol Device:R
- removed R15: 10K, symbol Device:R
- removed R24: 33, symbol Device:R
- removed R25: 470k, symbol Device:R
- removed R26: 390, symbol Device:R
- removed R27: 2.7k, symbol Device:R
- removed R3, R?: 27k, symbol Device:R
- removed R4: 8.2k, symbol Device:R
- removed R5: 100k, symbol Device:R
- removed R6: 1m, symbol Device:R
- removed SW1: RESET SWITCH, symbol Switch:SW_Push
- removed UIC44: MC14066, symbol Aamber:MC14066
- removed X1: 4MHz, symbol Device:Crystal
Connections:
- net labels removed: A0, A0-A15, A0-A9, A1, A10, A11, A12, A13, A14, A15, A2, A3, A4, A5, A6, A7, A8, A8-A15, A9, ASC, B0, B0-B7, B1, B2, B3, B4, B5, B6, B7, BLANK, C0, C0-C7, C1, C2, C3, C4, C5, C6, C7, CASSIN, CASSOUT, CHAR, CHAR-RAM, CHAR-ROM, CLR, CUA1, CUA2, CUB1, CUB2, D0, D0-D7, D1, D2, D3, D4, D5, D6, D7, D8, E, K0, K0-K3, K1, K2, K3, LOAD, MR, PA0, PA0-PA7, PA1, PA2, PA3, PA4, PA5, PA6, PA7, PAGE, PB0, PB0-PB7, PB1, PB2, PB3, PB4, PB5, PB6, PB7, PIA1, PIA2, R-W, R0, R0-R6, R1, R2, R3, R4, R5, R6, RAM1, RAM2, RAM3, RAM4, RESERVE, ROM1, ROM2, ROM3, SET, UA0, UA0-UA7, UA1, UA2, UA3, UA4, UA5, UA6, UA7, UB0, UB0-UB7, UB1, UB2, UB3, UB4, UB5, UB6, UB7, VAC, VID, VIDEO, X, ~DMA, ~E, ~FIRQ, ~H, ~HSYNC, ~IRQ, ~R-W, ~RESET, ~SET, ~VSYNC
- wire segments 1296 -> 136
Other:
- note added: "Power and bypassing\n"
- note removed: "50HERTZ"
