File: page-6-chargen.sch (KiCad schematic (older format))
At the start: 25 parts

Commit message: Fix missing IC numbers + Grid fixes
• IC numbers dissapeared in previous version. Fixed.
• Some grid issues. Fixed
• Some other small fixes
Parts:
- gave numbers to parts that had none: 21
Connections:
- net A10: no longer IC17.1, IC22.8
- net C2: now also IC37.12 (D03)
- net C3: no longer IC37.12 (D03)
- new net X: IC17.1, IC22.8
Changed lines of the file:
@@
 $EndDescr
 $Comp
-L Aamber:MC2114RAM IC?
+L Aamber:MC2114RAM IC37
 U 1 1 635D3D07
 P 11400 12350
-F 0 "IC?" H 11175 13020 50  0000 C CNN
+F 0 "IC37" H 11175 13020 50  0000 C CNN
 F 1 "MC2114RAM" H 11640 11695 50  0000 C CNN
 F 2 "" H 11400 12350 50  0001 C CNN
@@
 $EndComp
 $Comp
-L 74xx:74LS245 IC?
+L 74xx:74LS245 IC30
 U 1 1 635D3D0D
 P 8000 7050
-F 0 "IC?" H 7800 7850 50  0000 C CNN
+F 0 "IC30" H 7800 7850 50  0000 C CNN
 F 1 "74LS245" H 7700 7750 50  0000 C CNN
 F 2 "" H 8000 7050 50  0001 C CNN
@@
 $EndComp
 $Comp
-L Aamber:MC2114RAM IC?
+L Aamber:MC2114RAM IC32
 U 1 1 635D3D13
 P 13750 7150
-F 0 "IC?" H 13500 7800 50  0000 C CNN
+F 0 "IC32" H 13500 7800 50  0000 C CNN
 F 1 "MC2114RAM" H 14000 6500 50  0000 C CNN
 F 2 "" H 13750 7150 50  0001 C CNN
@@
 $EndComp
 $Comp
-L 74xx:74LS04 IC?
+L 74xx:74LS04 IC9
 U 4 1 635D3D19
 P 7950 4650
-F 0 "IC?" H 7950 4967 50  0000 C CNN
+F 0 "IC9" H 7950 4967 50  0000 C CNN
 F 1 "74LS04" H 7950 4876 50  0000 C CNN
 F 2 "" H 7950 4650 50  0001 C CNN
@@
 $EndComp
 $Comp
-L 74xx:74LS04 IC?
+L 74xx:74LS04 IC9
 U 2 1 635D3D1F
 P 7950 4100
-F 0 "IC?" H 7950 4417 50  0000 C CNN
+F 0 "IC9" H 7950 4417 50  0000 C CNN
 F 1 "74LS04" H 7950 4326 50  0000 C CNN
 F 2 "" H 7950 4100 50  0001 C CNN
@@
 $EndComp
 $Comp
-L 74xx:74LS20 IC?
+L 74xx:74LS20 IC22
 U 2 1 635D3D25
 P 8900 4500
-F 0 "IC?" H 8900 4875 50  0000 C CNN
+F 0 "IC22" H 8900 4875 50  0000 C CNN
 F 1 "74LS20" H 8900 4784 50  0000 C CNN
 F 2 "" H 8900 4500 50  0001 C CNN
@@
 $EndComp
 $Comp
-L 74xx:74LS08 IC?
+L 74xx:74LS08 IC17
 U 1 1 635D3D2B
 P 9850 4600
-F 0 "IC?" H 9850 4925 50  0000 C CNN
+F 0 "IC17" H 9850 4925 50  0000 C CNN
 F 1 "74LS08" H 9850 4834 50  0000 C CNN
 F 2 "" H 9850 4600 50  0001 C CNN
@@
 	14900 7250 14250 7250
 $Comp
-L Aamber:MC2114RAM IC?
+L Aamber:MC2114RAM IC31
 U 1 1 635D3D32
 P 11350 7100
-F 0 "IC?" H 11100 7750 50  0000 C CNN
+F 0 "IC31" H 11100 7750 50  0000 C CNN
 F 1 "MC2114RAM" H 11600 6450 50  0000 C CNN
 F 2 "" H 11350 7100 50  0001 C CNN
@@
 	8250 3050 8450 3050
 $Comp
-L 74xx:74LS32 IC?
+L 74xx:74LS32 IC2
 U 4 1 635D3D73
 P 7950 3050
-F 0 "IC?" H 7950 3375 50  0000 C CNN
+F 0 "IC2" H 7950 3375 50  0000 C CNN
 F 1 "74LS32" H 7950 3284 50  0000 C CNN
 F 2 "" H 7950 3050 50  0001 C CNN
@@
 $EndComp
 $Comp
-L 74xx:74LS04 IC?
+L 74xx:74LS04 IC9
 U 5 1 635D3D79
 P 8900 3050
-F 0 "IC?" H 8900 3367 50  0000 C CNN
+F 0 "IC9" H 8900 3367 50  0000 C CNN
 F 1 "74LS04" H 8900 3276 50  0000 C CNN
 F 2 "" H 8900 3050 50  0001 C CNN
@@
 $EndComp
 $Comp
-L 74xx:74LS00 IC?
+L 74xx:74LS00 IC3
 U 2 1 635D3D7F
 P 10050 3150
-F 0 "IC?" H 10050 3475 50  0000 C CNN
+F 0 "IC3" H 10050 3475 50  0000 C CNN
 F 1 "74LS00" H 10050 3384 50  0000 C CNN
 F 2 "" H 10050 3150 50  0001 C CNN
@@
 P 8500 10050
 F 0 "#PWR?" H 8500 9900 50  0001 C CNN
-F 1 "+5V" H 8515 10178 50  0000 L CNN
+F 1 "+5V" V 8515 10178 50  0000 L CNN
 F 2 "" H 8500 10050 50  0001 C CNN
 F 3 "" H 8500 10050 50  0001 C CNN
@@
 	8700 10050 8500 10050
 $Comp
-L 74xx:74LS86 IC?
+L 74xx:74LS86 IC33
 U 2 1 635D3E5A
 P 9000 9950
-F 0 "IC?" H 9000 9633 50  0000 C CNN
+F 0 "IC33" H 9000 9633 50  0000 C CNN
 F 1 "74LS86" H 9000 9724 50  0000 C CNN
 F 2 "" H 9000 9950 50  0001 C CNN
@@
 $EndComp
 $Comp
-L 74xx:74LS32 IC?
+L 74xx:74LS32 IC2
 U 3 1 635D3E60
 P 15150 9750
-F 0 "IC?" H 15150 9433 50  0000 C CNN
+F 0 "IC2" H 15150 9433 50  0000 C CNN
 F 1 "74LS32" H 15150 9524 50  0000 C CNN
 F 2 "" H 15150 9750 50  0001 C CNN
@@
 	15450 9850 16050 9850
 $Comp
-L 74xx:74LS08 IC?
+L 74xx:74LS08 IC17
 U 2 1 635D3E67
 P 10600 4700
-F 0 "IC?" H 10600 5025 50  0000 C CNN
+F 0 "IC17" H 10600 5025 50  0000 C CNN
 F 1 "74LS08" H 10600 4934 50  0000 C CNN
 F 2 "" H 10600 4700 50  0001 C CNN
@@
 A9
 Text GLabel 13700 5500 2    50   Input ~ 0
-A0-A9
+A0-A15
 Wire Wire Line
 	8450 3400 15700 3400
@@
 	15450 9650 15700 9650
 $Comp
-L Aamber:MC66710 IC?
+L Aamber:MC66710 IC36
 U 1 1 635D3EBE
 P 8650 12000
-F 0 "IC?" H 8445 13310 50  0000 C CNN
+F 0 "IC36" H 8445 13310 50  0000 C CNN
 F 1 "MC66710" H 8365 13200 50  0000 C CNN
 F 2 "" H 8400 11800 50  0001 C CNN
@@
 Connection ~ 10000 11850
 $Comp
-L Aamber:MC2114RAM IC?
+L Aamber:MC2114RAM IC38
 U 1 1 635D3ED2
 P 13700 12350
-F 0 "IC?" H 13495 13005 50  0000 C CNN
+F 0 "IC38" H 13495 13005 50  0000 C CNN
 F 1 "MC2114RAM" H 13940 11700 50  0000 C CNN
 F 2 "" H 13700 12350 50  0001 C CNN
@@
 	11900 9750 11900 10850
 $Comp
-L Aamber:MC2114RAM IC?
+L Aamber:MC2114RAM IC34
 U 1 1 635D3EF4
 P 11400 9650
-F 0 "IC?" H 11185 10325 50  0000 C CNN
+F 0 "IC34" H 11185 10325 50  0000 C CNN
 F 1 "MC2114RAM" H 11630 9005 50  0000 C CNN
 F 2 "" H 11400 9650 50  0001 C CNN
@@
 	14200 9750 14700 9750
 $Comp
-L Aamber:MC2114RAM IC?
+L Aamber:MC2114RAM IC35
 U 1 1 635D3F80
 P 13700 9650
-F 0 "IC?" H 13475 10310 50  0000 C CNN
+F 0 "IC35" H 13475 10310 50  0000 C CNN
 F 1 "MC2114RAM" H 13950 9005 50  0000 C CNN
 F 2 "" H 13700 9650 50  0001 C CNN
@@
 C3
 Text Label 11900 12050 0    50   ~ 0
-C3
+C2
 Text Label 11900 11950 0    50   ~ 0
 C1
@@
 	7800 10900 7900 11000
 $Comp
-L Device:R R?
+L Device:R R16
 U 1 1 635D3FDE
 P 7250 8900
-F 0 "R?" V 7350 9000 50  0000 R CNN
+F 0 "R16" V 7350 9000 50  0000 R CNN
 F 1 "1k" V 7150 9000 50  0000 R CNN
 F 2 "" V 7180 8900 50  0001 C CNN
@@
 $EndComp
 $Comp
-L Device:R R?
+L Device:R R19
 U 1 1 635D3FE4
 P 7250 9800
-F 0 "R?" V 7350 9900 50  0000 R CNN
+F 0 "R19" V 7350 9900 50  0000 R CNN
 F 1 "1k" V 7150 9900 50  0000 R CNN
 F 2 "" V 7180 9800 50  0001 C CNN
@@
 $EndComp
 $Comp
-L Device:R R?
+L Device:R R17
 U 1 1 635D3FEA
 P 7250 9200
-F 0 "R?" V 7350 9300 50  0000 R CNN
+F 0 "R17" V 7350 9300 50  0000 R CNN
 F 1 "1k" V 7150 9300 50  0000 R CNN
 F 2 "" V 7180 9200 50  0001 C CNN
@@
 $EndComp
 $Comp
-L Device:R R?
+L Device:R R18
 U 1 1 635D3FF0
 P 7250 9500
-F 0 "R?" V 7350 9600 50  0000 R CNN
+F 0 "R18" V 7350 9600 50  0000 R CNN
 F 1 "1k" V 7150 9600 50  0000 R CNN
 F 2 "" V 7180 9500 50  0001 C CNN
@@
 	7100 10400 6950 10400
 $Comp
-L Device:R R?
+L Device:R R22
 U 1 1 635D401D
 P 7250 10700
-F 0 "R?" V 7350 10800 50  0000 R CNN
+F 0 "R22" V 7350 10800 50  0000 R CNN
 F 1 "1k" V 7150 10800 50  0000 R CNN
 F 2 "" V 7180 10700 50  0001 C CNN
@@
 $EndComp
 $Comp
-L Device:R R?
+L Device:R R21
 U 1 1 635D4023
 P 7250 10400
-F 0 "R?" V 7350 10500 50  0000 R CNN
+F 0 "R21" V 7350 10500 50  0000 R CNN
 F 1 "1k" V 7150 10500 50  0000 R CNN
 F 2 "" V 7180 10400 50  0001 C CNN
@@
 	7100 10100 6950 10100
 $Comp
-L Device:R R?
+L Device:R R20
 U 1 1 635D4032
 P 7250 10100
-F 0 "R?" V 7350 10200 50  0000 R CNN
+F 0 "R20" V 7350 10200 50  0000 R CNN
 F 1 "1k" V 7150 10200 50  0000 R CNN
 F 2 "" V 7180 10100 50  0001 C CNN
@@
 B0-B7
 Text Label 13350 5500 0    50   ~ 0
-A0-A9
+A0-A15
 Text Label 7400 5900 0    50   ~ 0
 D0-D7
@@
 X
 Text Label 6450 5000 0    50   ~ 0
-X
+A10
 Text Label 6450 4650 0    50   ~ 0
 ROM1
