File: page-1-video-timing.sch (KiCad schematic (older format))
At the start: 18 parts, among them IC1 74LS14, IC2 74LS32, IC3 74LS00, IC4 74LS21, IC5 74LS123, IC6 74LS74, IC7 74LS93, IC8 74LS93, IC9 74LS04

Commit message: Review and clean up page 1
Parts:
- renumbered IC6 to IC46
Other:
- note added: "Created: PL, 2/27/2020\nReviewed: DF, 4/15/2020"
- moved on the sheet: C1, C2, D1, D2, IC1C, IC2B, IC3C, IC46A, IC4A, IC5A, IC5B, IC6A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
